File: extra/vfd.sch (KiCad schematic (older format))
At the start: 42 parts, among them P10 GU128x64E-U100, P11 gui140x16j-7002, P12 digital_in, P13 digital_out, U3 74LS125, U4 74LS125, U5 74LS125, U6 74LS125, U7 74LS125, U8 74LS245

Commit message: starting pcb layout a little
Parts:
- D10, D11, D12, D13, D2, D3, D4, D5, D6, D7, D8, D9: footprint (none) -> Diodes_ThroughHole:Diode_DO-41_SOD81_Horizontal_RM10
- P10: footprint (none) -> Pin_Headers:Pin_Header_Straight_1x16_Pitch2.54mm
- P11: footprint (none) -> Pin_Headers:Pin_Header_Straight_2x06_Pitch2.54mm
- P12: footprint (none) -> Pin_Headers:Pin_Header_Straight_1x07_Pitch2.54mm
- P13: footprint (none) -> Pin_Headers:Pin_Header_Straight_1x08_Pitch2.54mm
- U3, U4, U5, U6, U7, U8: footprint (none) -> Housings_DIP:DIP-14_W7.62mm_LongPads
Changed lines of the file:
@@
 F 0 "P11" H 1500 1350 50  0000 C CNN
 F 1 "gui140x16j-7002" V 1500 950 50  0000 C CNN
-F 2 "" H 1500 -250 50  0001 C CNN
+F 2 "Pin_Headers:Pin_Header_Straight_2x06_Pitch2.54mm" H 1500 -250 50  0001 C CNN
 F 3 "" H 1500 -250 50  0000 C CNN
 	1    1500 950
@@
 F 0 "U3" H 1700 3400 50  0000 L BNN
 F 1 "74LS125" H 1750 3150 50  0000 L TNN
-F 2 "" H 1700 3300 50  0001 C CNN
+F 2 "Housings_DIP:DIP-14_W7.62mm_LongPads" H 1700 3300 50  0001 C CNN
 F 3 "" H 1700 3300 50  0000 C CNN
 	1    1700 3300
@@
 F 0 "U3" H 1700 3950 50  0000 L BNN
 F 1 "74LS125" H 1750 3700 50  0000 L TNN
-F 2 "" H 1700 3850 50  0001 C CNN
+F 2 "Housings_DIP:DIP-14_W7.62mm_LongPads" H 1700 3850 50  0001 C CNN
 F 3 "" H 1700 3850 50  0000 C CNN
 	2    1700 3850
@@
 F 0 "U3" H 1700 4550 50  0000 L BNN
 F 1 "74LS125" H 1750 4300 50  0000 L TNN
-F 2 "" H 1700 4450 50  0001 C CNN
+F 2 "Housings_DIP:DIP-14_W7.62mm_LongPads" H 1700 4450 50  0001 C CNN
 F 3 "" H 1700 4450 50  0000 C CNN
 	3    1700 4450
@@
 F 0 "U3" H 1700 5050 50  0000 L BNN
 F 1 "74LS125" H 1750 4800 50  0000 L TNN
-F 2 "" H 1700 4950 50  0001 C CNN
+F 2 "Housings_DIP:DIP-14_W7.62mm_LongPads" H 1700 4950 50  0001 C CNN
 F 3 "" H 1700 4950 50  0000 C CNN
 	4    1700 4950
@@
 F 0 "U4" H 1700 5700 50  0000 L BNN
 F 1 "74LS125" H 1750 5450 50  0000 L TNN
-F 2 "" H 1700 5600 50  0001 C CNN
+F 2 "Housings_DIP:DIP-14_W7.62mm_LongPads" H 1700 5600 50  0001 C CNN
 F 3 "" H 1700 5600 50  0000 C CNN
 	1    1700 5600
@@
 F 0 "U4" H 1700 6250 50  0000 L BNN
 F 1 "74LS125" H 1750 6000 50  0000 L TNN
-F 2 "" H 1700 6150 50  0001 C CNN
+F 2 "Housings_DIP:DIP-14_W7.62mm_LongPads" H 1700 6150 50  0001 C CNN
 F 3 "" H 1700 6150 50  0000 C CNN
 	2    1700 6150
@@
 F 0 "U4" H 1700 6850 50  0000 L BNN
 F 1 "74LS125" H 1750 6600 50  0000 L TNN
-F 2 "" H 1700 6750 50  0001 C CNN
+F 2 "Housings_DIP:DIP-14_W7.62mm_LongPads" H 1700 6750 50  0001 C CNN
 F 3 "" H 1700 6750 50  0000 C CNN
 	3    1700 6750
@@
 F 0 "U4" H 1700 7350 50  0000 L BNN
 F 1 "74LS125" H 1750 7100 50  0000 L TNN
-F 2 "" H 1700 7250 50  0001 C CNN
+F 2 "Housings_DIP:DIP-14_W7.62mm_LongPads" H 1700 7250 50  0001 C CNN
 F 3 "" H 1700 7250 50  0000 C CNN
 	4    1700 7250
@@
 F 0 "U5" H 5600 3300 50  0000 L BNN
 F 1 "74LS125" H 5650 3050 50  0000 L TNN
-F 2 "" H 5600 3200 50  0001 C CNN
+F 2 "Housings_DIP:DIP-14_W7.62mm_LongPads" H 5600 3200 50  0001 C CNN
 F 3 "" H 5600 3200 50  0000 C CNN
 	1    5600 3200
@@
 F 0 "U5" H 5600 3850 50  0000 L BNN
 F 1 "74LS125" H 5650 3600 50  0000 L TNN
-F 2 "" H 5600 3750 50  0001 C CNN
+F 2 "Housings_DIP:DIP-14_W7.62mm_LongPads" H 5600 3750 50  0001 C CNN
 F 3 "" H 5600 3750 50  0000 C CNN
 	2    5600 3750
@@
 F 0 "U5" H 5600 4450 50  0000 L BNN
 F 1 "74LS125" H 5650 4200 50  0000 L TNN
-F 2 "" H 5600 4350 50  0001 C CNN
+F 2 "Housings_DIP:DIP-14_W7.62mm_LongPads" H 5600 4350 50  0001 C CNN
 F 3 "" H 5600 4350 50  0000 C CNN
 	3    5600 4350
@@
 F 0 "U5" H 5600 4950 50  0000 L BNN
 F 1 "74LS125" H 5650 4700 50  0000 L TNN
-F 2 "" H 5600 4850 50  0001 C CNN
+F 2 "Housings_DIP:DIP-14_W7.62mm_LongPads" H 5600 4850 50  0001 C CNN
 F 3 "" H 5600 4850 50  0000 C CNN
 	4    5600 4850
@@
 F 0 "U6" H 5600 5600 50  0000 L BNN
 F 1 "74LS125" H 5650 5350 50  0000 L TNN
-F 2 "" H 5600 5500 50  0001 C CNN
+F 2 "Housings_DIP:DIP-14_W7.62mm_LongPads" H 5600 5500 50  0001 C CNN
 F 3 "" H 5600 5500 50  0000 C CNN
 	1    5600 5500
@@
 F 0 "U6" H 5600 6150 50  0000 L BNN
 F 1 "74LS125" H 5650 5900 50  0000 L TNN
-F 2 "" H 5600 6050 50  0001 C CNN
+F 2 "Housings_DIP:DIP-14_W7.62mm_LongPads" H 5600 6050 50  0001 C CNN
 F 3 "" H 5600 6050 50  0000 C CNN
 	2    5600 6050
@@
 F 0 "U6" H 5600 6750 50  0000 L BNN
 F 1 "74LS125" H 5650 6500 50  0000 L TNN
-F 2 "" H 5600 6650 50  0001 C CNN
+F 2 "Housings_DIP:DIP-14_W7.62mm_LongPads" H 5600 6650 50  0001 C CNN
 F 3 "" H 5600 6650 50  0000 C CNN
 	3    5600 6650
@@
 F 0 "U6" H 5600 7250 50  0000 L BNN
 F 1 "74LS125" H 5650 7000 50  0000 L TNN
-F 2 "" H 5600 7150 50  0001 C CNN
+F 2 "Housings_DIP:DIP-14_W7.62mm_LongPads" H 5600 7150 50  0001 C CNN
 F 3 "" H 5600 7150 50  0000 C CNN
 	4    5600 7150
@@
 F 0 "U8" H 9750 2375 50  0000 L BNN
 F 1 "74LS245" H 9700 1225 50  0000 L TNN
-F 2 "" H 9650 1800 50  0001 C CNN
+F 2 "Housings_DIP:DIP-14_W7.62mm_LongPads" H 9650 1800 50  0001 C CNN
 F 3 "" H 9650 1800 50  0000 C CNN
 	1    9650 1800
@@
 F 0 "P10" H -250 2650 50  0000 C CNN
 F 1 "GU128x64E-U100" V -150 1800 50  0000 C CNN
-F 2 "" H -250 1800 50  0001 C CNN
+F 2 "Pin_Headers:Pin_Header_Straight_1x16_Pitch2.54mm" H -250 1800 50  0001 C CNN
 F 3 "" H -250 1800 50  0000 C CNN
 	1    -250 1800
@@
 F 0 "U7" H 9200 4600 50  0000 L BNN
 F 1 "74LS125" H 9250 4350 50  0000 L TNN
-F 2 "" H 9200 4500 50  0001 C CNN
+F 2 "Housings_DIP:DIP-14_W7.62mm_LongPads" H 9200 4500 50  0001 C CNN
 F 3 "" H 9200 4500 50  0000 C CNN
 	1    9200 4500
@@
 F 0 "U7" H 9200 5150 50  0000 L BNN
 F 1 "74LS125" H 9250 4900 50  0000 L TNN
-F 2 "" H 9200 5050 50  0001 C CNN
+F 2 "Housings_DIP:DIP-14_W7.62mm_LongPads" H 9200 5050 50  0001 C CNN
 F 3 "" H 9200 5050 50  0000 C CNN
 	2    9200 5050
@@
 F 0 "U7" H 9200 5750 50  0000 L BNN
 F 1 "74LS125" H 9250 5500 50  0000 L TNN
-F 2 "" H 9200 5650 50  0001 C CNN
+F 2 "Housings_DIP:DIP-14_W7.62mm_LongPads" H 9200 5650 50  0001 C CNN
 F 3 "" H 9200 5650 50  0000 C CNN
 	3    9200 5650
@@
 F 0 "U7" H 9200 6250 50  0000 L BNN
 F 1 "74LS125" H 9250 6000 50  0000 L TNN
-F 2 "" H 9200 6150 50  0001 C CNN
+F 2 "Housings_DIP:DIP-14_W7.62mm_LongPads" H 9200 6150 50  0001 C CNN
 F 3 "" H 9200 6150 50  0000 C CNN
 	4    9200 6150
@@
 F 0 "P13" H 6400 2100 50  0000 C CNN
 F 1 "digital_out" V 6500 1650 50  0000 C CNN
-F 2 "" H 6400 1650 50  0001 C CNN
+F 2 "Pin_Headers:Pin_Header_Straight_1x08_Pitch2.54mm" H 6400 1650 50  0001 C CNN
 F 3 "" H 6400 1650 50  0000 C CNN
 	1    6400 1650
@@
 F 0 "D13" H 5400 2250 50  0000 C CNN
 F 1 "D" H 5400 2050 50  0000 C CNN
-F 2 "" H 5400 2150 50  0001 C CNN
+F 2 "Diodes_ThroughHole:Diode_DO-41_SOD81_Horizontal_RM10" H 5400 2150 50  0001 C CNN
 F 3 "" H 5400 2150 50  0000 C CNN
 	1    5400 2150
@@
 F 0 "D12" H 5400 1150 50  0000 C CNN
 F 1 "D" H 5400 950 50  0000 C CNN
-F 2 "" H 5400 1050 50  0001 C CNN
+F 2 "Diodes_ThroughHole:Diode_DO-41_SOD81_Horizontal_RM10" H 5400 1050 50  0001 C CNN
 F 3 "" H 5400 1050 50  0000 C CNN
 	1    5400 1050
@@
 F 0 "D10" H 5300 1150 50  0000 C CNN
 F 1 "D" H 5300 950 50  0000 C CNN
-F 2 "" H 5300 1050 50  0001 C CNN
+F 2 "Diodes_ThroughHole:Diode_DO-41_SOD81_Horizontal_RM10" H 5300 1050 50  0001 C CNN
 F 3 "" H 5300 1050 50  0000 C CNN
 	1    5300 1050
@@
 F 0 "D8" H 5200 1150 50  0000 C CNN
 F 1 "D" H 5200 950 50  0000 C CNN
-F 2 "" H 5200 1050 50  0001 C CNN
+F 2 "Diodes_ThroughHole:Diode_DO-41_SOD81_Horizontal_RM10" H 5200 1050 50  0001 C CNN
 F 3 "" H 5200 1050 50  0000 C CNN
 	1    5200 1050
@@
 F 0 "D6" H 5100 1150 50  0000 C CNN
 F 1 "D" H 5100 950 50  0000 C CNN
-F 2 "" H 5100 1050 50  0001 C CNN
+F 2 "Diodes_ThroughHole:Diode_DO-41_SOD81_Horizontal_RM10" H 5100 1050 50  0001 C CNN
 F 3 "" H 5100 1050 50  0000 C CNN
 	1    5100 1050
@@
 F 0 "D4" H 5000 1150 50  0000 C CNN
 F 1 "D" H 5000 950 50  0000 C CNN
-F 2 "" H 5000 1050 50  0001 C CNN
+F 2 "Diodes_ThroughHole:Diode_DO-41_SOD81_Horizontal_RM10" H 5000 1050 50  0001 C CNN
 F 3 "" H 5000 1050 50  0000 C CNN
 	1    5000 1050
@@
 F 0 "D2" H 4900 1150 50  0000 C CNN
 F 1 "D" H 4900 950 50  0000 C CNN
-F 2 "" H 4900 1050 50  0001 C CNN
+F 2 "Diodes_ThroughHole:Diode_DO-41_SOD81_Horizontal_RM10" H 4900 1050 50  0001 C CNN
 F 3 "" H 4900 1050 50  0000 C CNN
 	1    4900 1050
@@
 F 0 "D11" H 5300 2250 50  0000 C CNN
 F 1 "D" H 5300 2050 50  0000 C CNN
-F 2 "" H 5300 2150 50  0001 C CNN
+F 2 "Diodes_ThroughHole:Diode_DO-41_SOD81_Horizontal_RM10" H 5300 2150 50  0001 C CNN
 F 3 "" H 5300 2150 50  0000 C CNN
 	1    5300 2150
@@
 F 0 "D9" H 5200 2250 50  0000 C CNN
 F 1 "D" H 5200 2050 50  0000 C CNN
-F 2 "" H 5200 2150 50  0001 C CNN
+F 2 "Diodes_ThroughHole:Diode_DO-41_SOD81_Horizontal_RM10" H 5200 2150 50  0001 C CNN
 F 3 "" H 5200 2150 50  0000 C CNN
 	1    5200 2150
@@
 F 0 "D7" H 5100 2250 50  0000 C CNN
 F 1 "D" H 5100 2050 50  0000 C CNN
-F 2 "" H 5100 2150 50  0001 C CNN
+F 2 "Diodes_ThroughHole:Diode_DO-41_SOD81_Horizontal_RM10" H 5100 2150 50  0001 C CNN
 F 3 "" H 5100 2150 50  0000 C CNN
 	1    5100 2150
@@
 F 0 "D5" H 5000 2250 50  0000 C CNN
 F 1 "D" H 5000 2050 50  0000 C CNN
-F 2 "" H 5000 2150 50  0001 C CNN
+F 2 "Diodes_ThroughHole:Diode_DO-41_SOD81_Horizontal_RM10" H 5000 2150 50  0001 C CNN
 F 3 "" H 5000 2150 50  0000 C CNN
 	1    5000 2150
@@
 F 0 "D3" H 4900 2250 50  0000 C CNN
 F 1 "D" H 4900 2050 50  0000 C CNN
-F 2 "" H 4900 2150 50  0001 C CNN
+F 2 "Diodes_ThroughHole:Diode_DO-41_SOD81_Horizontal_RM10" H 4900 2150 50  0001 C CNN
 F 3 "" H 4900 2150 50  0000 C CNN
 	1    4900 2150
@@
 F 0 "P12" H 3050 1950 50  0000 C CNN
 F 1 "digital_in" V 3150 1550 50  0000 C CNN
-F 2 "" H 3050 1550 50  0001 C CNN
+F 2 "Pin_Headers:Pin_Header_Straight_1x07_Pitch2.54mm" H 3050 1550 50  0001 C CNN
 F 3 "" H 3050 1550 50  0000 C CNN
 	1    3050 1550

Commit message: moving along, still no idea why 5v is hooked to 3.3v
Parts:
- U8: footprint Housings_DIP:DIP-14_W7.62mm_LongPads -> Housings_DIP:DIP-20_W7.62mm_LongPads
Changed lines of the file:
@@
 LIBS:contrib
 LIBS:valves
+LIBS:xnorman
 LIBS:bela-extra-cache
 EELAYER 25 0
@@
 5v
 $Comp
-L GND #PWR017
+L GND #PWR018
 U 1 1 58578899
 P 750 650
-F 0 "#PWR017" H 750 400 50  0001 C CNN
+F 0 "#PWR018" H 750 400 50  0001 C CNN
 F 1 "GND" H 750 500 50  0000 C CNN
 F 2 "" H 750 650 50  0000 C CNN
@@
 vfdD7
 $Comp
-L GND #PWR018
+L GND #PWR019
 U 1 1 5857965E
 P 1350 7050
-F 0 "#PWR018" H 1350 6800 50  0001 C CNN
+F 0 "#PWR019" H 1350 6800 50  0001 C CNN
 F 1 "GND" H 1350 6900 50  0000 C CNN
 F 2 "" H 1350 7050 50  0000 C CNN
@@
 $EndComp
 $Comp
-L GND #PWR019
+L GND #PWR020
 U 1 1 585796B9
 P 1350 6450
-F 0 "#PWR019" H 1350 6200 50  0001 C CNN
+F 0 "#PWR020" H 1350 6200 50  0001 C CNN
 F 1 "GND" H 1350 6300 50  0000 C CNN
 F 2 "" H 1350 6450 50  0000 C CNN
@@
 $EndComp
 $Comp
-L GND #PWR020
+L GND #PWR021
 U 1 1 585796DF
 P 1350 5900
-F 0 "#PWR020" H 1350 5650 50  0001 C CNN
+F 0 "#PWR021" H 1350 5650 50  0001 C CNN
 F 1 "GND" H 1350 5750 50  0000 C CNN
 F 2 "" H 1350 5900 50  0000 C CNN
@@
 $EndComp
 $Comp
-L GND #PWR021
+L GND #PWR022
 U 1 1 5857970E
 P 1350 5250
-F 0 "#PWR021" H 1350 5000 50  0001 C CNN
+F 0 "#PWR022" H 1350 5000 50  0001 C CNN
 F 1 "GND" H 1350 5100 50  0000 C CNN
 F 2 "" H 1350 5250 50  0000 C CNN
@@
 $EndComp
 $Comp
-L GND #PWR022
+L GND #PWR023
 U 1 1 58579734
 P 1350 4750
-F 0 "#PWR022" H 1350 4500 50  0001 C CNN
+F 0 "#PWR023" H 1350 4500 50  0001 C CNN
 F 1 "GND" H 1350 4600 50  0000 C CNN
 F 2 "" H 1350 4750 50  0000 C CNN
@@
 $EndComp
 $Comp
-L GND #PWR023
+L GND #PWR024
 U 1 1 58579763
 P 1350 4150
-F 0 "#PWR023" H 1350 3900 50  0001 C CNN
+F 0 "#PWR024" H 1350 3900 50  0001 C CNN
 F 1 "GND" H 1350 4000 50  0000 C CNN
 F 2 "" H 1350 4150 50  0000 C CNN
@@
 $EndComp
 $Comp
-L GND #PWR024
+L GND #PWR025
 U 1 1 58579789
 P 1350 3600
-F 0 "#PWR024" H 1350 3350 50  0001 C CNN
+F 0 "#PWR025" H 1350 3350 50  0001 C CNN
 F 1 "GND" H 1350 3450 50  0000 C CNN
 F 2 "" H 1350 3600 50  0000 C CNN
@@
 vfdCS2
 $Comp
-L GND #PWR025
+L GND #PWR026
 U 1 1 58579E92
 P 5200 5150
-F 0 "#PWR025" H 5200 4900 50  0001 C CNN
+F 0 "#PWR026" H 5200 4900 50  0001 C CNN
 F 1 "GND" H 5200 5000 50  0000 C CNN
 F 2 "" H 5200 5150 50  0000 C CNN
@@
 $EndComp
 $Comp
-L GND #PWR026
+L GND #PWR027
 U 1 1 58579E98
 P 5200 4650
-F 0 "#PWR026" H 5200 4400 50  0001 C CNN
+F 0 "#PWR027" H 5200 4400 50  0001 C CNN
 F 1 "GND" H 5200 4500 50  0000 C CNN
 F 2 "" H 5200 4650 50  0000 C CNN
@@
 $EndComp
 $Comp
-L GND #PWR027
+L GND #PWR028
 U 1 1 58579E9E
 P 5200 4050
-F 0 "#PWR027" H 5200 3800 50  0001 C CNN
+F 0 "#PWR028" H 5200 3800 50  0001 C CNN
 F 1 "GND" H 5200 3900 50  0000 C CNN
 F 2 "" H 5200 4050 50  0000 C CNN
@@
 $EndComp
 $Comp
-L GND #PWR028
+L GND #PWR029
 U 1 1 58579EA4
 P 5200 3500
-F 0 "#PWR028" H 5200 3250 50  0001 C CNN
+F 0 "#PWR029" H 5200 3250 50  0001 C CNN
 F 1 "GND" H 5200 3350 50  0000 C CNN
 F 2 "" H 5200 3500 50  0000 C CNN
@@
 moddigout4
 $Comp
-L GND #PWR029
+L GND #PWR030
 U 1 1 5857A461
 P 5200 7450
-F 0 "#PWR029" H 5200 7200 50  0001 C CNN
+F 0 "#PWR030" H 5200 7200 50  0001 C CNN
 F 1 "GND" H 5200 7300 50  0000 C CNN
 F 2 "" H 5200 7450 50  0000 C CNN
@@
 $EndComp
 $Comp
-L GND #PWR030
+L GND #PWR031
 U 1 1 5857A467
 P 5200 6950
-F 0 "#PWR030" H 5200 6700 50  0001 C CNN
+F 0 "#PWR031" H 5200 6700 50  0001 C CNN
 F 1 "GND" H 5200 6800 50  0000 C CNN
 F 2 "" H 5200 6950 50  0000 C CNN
@@
 $EndComp
 $Comp
-L GND #PWR031
+L GND #PWR032
 U 1 1 5857A46D
 P 5200 6350
-F 0 "#PWR031" H 5200 6100 50  0001 C CNN
+F 0 "#PWR032" H 5200 6100 50  0001 C CNN
 F 1 "GND" H 5200 6200 50  0000 C CNN
 F 2 "" H 5200 6350 50  0000 C CNN
@@
 $EndComp
 $Comp
-L GND #PWR032
+L GND #PWR033
 U 1 1 5857A473
 P 5200 5800
-F 0 "#PWR032" H 5200 5550 50  0001 C CNN
+F 0 "#PWR033" H 5200 5550 50  0001 C CNN
 F 1 "GND" H 5200 5650 50  0000 C CNN
 F 2 "" H 5200 5800 50  0000 C CNN
@@
 	0    1    1    0
 $EndComp
-$Comp
-L 74LS245 U8
-U 1 1 5857A66B
-P 9650 1800
-F 0 "U8" H 9750 2375 50  0000 L BNN
-F 1 "74LS245" H 9700 1225 50  0000 L TNN
-F 2 "Housings_DIP:DIP-14_W7.62mm_LongPads" H 9650 1800 50  0001 C CNN
-F 3 "" H 9650 1800 50  0000 C CNN
-	1    9650 1800
-	1    0    0    -1
-$EndComp
 Text GLabel 9650 1050 1    60   Input ~ 0
 3.3v
 $Comp
-L GND #PWR033
+L GND #PWR034
 U 1 1 5857B8FE
 P 9650 2550
-F 0 "#PWR033" H 9650 2300 50  0001 C CNN
+F 0 "#PWR034" H 9650 2300 50  0001 C CNN
 F 1 "GND" H 9650 2400 50  0000 C CNN
 F 2 "" H 9650 2550 50  0000 C CNN
@@
 	5200 7450 5600 7450
 Wire Wire Line
-	9650 1050 9650 1250
-Wire Wire Line
 	9650 2350 9650 2550
 Wire Wire Line
@@
 $EndComp
 $Comp
-L GND #PWR034
+L GND #PWR035
 U 1 1 586B1181
 P -700 950
-F 0 "#PWR034" H -700 700 50  0001 C CNN
+F 0 "#PWR035" H -700 700 50  0001 C CNN
 F 1 "GND" H -700 800 50  0000 C CNN
 F 2 "" H -700 950 50  0000 C CNN
@@
 vfdE
 $Comp
-L GND #PWR035
+L GND #PWR036
 U 1 1 586B61FC
 P 8800 6450
-F 0 "#PWR035" H 8800 6200 50  0001 C CNN
+F 0 "#PWR036" H 8800 6200 50  0001 C CNN
 F 1 "GND" H 8800 6300 50  0000 C CNN
 F 2 "" H 8800 6450 50  0000 C CNN
@@
 $EndComp
 $Comp
-L GND #PWR036
+L GND #PWR037
 U 1 1 586B6202
 P 8800 5950
-F 0 "#PWR036" H 8800 5700 50  0001 C CNN
+F 0 "#PWR037" H 8800 5700 50  0001 C CNN
 F 1 "GND" H 8800 5800 50  0000 C CNN
 F 2 "" H 8800 5950 50  0000 C CNN
@@
 $EndComp
 $Comp
-L GND #PWR037
+L GND #PWR038
 U 1 1 586B6208
 P 8800 5350
-F 0 "#PWR037" H 8800 5100 50  0001 C CNN
+F 0 "#PWR038" H 8800 5100 50  0001 C CNN
 F 1 "GND" H 8800 5200 50  0000 C CNN
 F 2 "" H 8800 5350 50  0000 C CNN
@@
 $EndComp
 $Comp
-L GND #PWR038
+L GND #PWR039
 U 1 1 586B620E
 P 8800 4800
-F 0 "#PWR038" H 8800 4550 50  0001 C CNN
+F 0 "#PWR039" H 8800 4550 50  0001 C CNN
 F 1 "GND" H 8800 4650 50  0000 C CNN
 F 2 "" H 8800 4800 50  0000 C CNN
@@
 	3250 1750 4150 1750
 $Comp
-L GND #PWR039
+L GND #PWR040
 U 1 1 586B38A8
 P 3250 2150
-F 0 "#PWR039" H 3250 1900 50  0001 C CNN
+F 0 "#PWR040" H 3250 1900 50  0001 C CNN
 F 1 "GND" H 3250 2000 50  0000 C CNN
 F 2 "" H 3250 2150 50  0000 C CNN
@@
 	6700 2050 6850 2050
 $Comp
-L GND #PWR040
+L GND #PWR041
 U 1 1 586B6695
 P 6600 2200
-F 0 "#PWR040" H 6600 1950 50  0001 C CNN
+F 0 "#PWR041" H 6600 1950 50  0001 C CNN
 F 1 "GND" H 6600 2050 50  0000 C CNN
 F 2 "" H 6600 2200 50  0000 C CNN
@@
 Connection ~ 5400 1250
 $Comp
-L GND #PWR041
+L GND #PWR042
 U 1 1 586B8342
 P 5400 2350
-F 0 "#PWR041" H 5400 2100 50  0001 C CNN
+F 0 "#PWR042" H 5400 2100 50  0001 C CNN
 F 1 "GND" H 5400 2200 50  0000 C CNN
 F 2 "" H 5400 2350 50  0000 C CNN
@@
 digital input protection, needed if we're using level shifter???
 $Comp
-L GND #PWR042
+L GND #PWR043
 U 1 1 586B5219
 P 4350 2550
-F 0 "#PWR042" H 4350 2300 50  0001 C CNN
+F 0 "#PWR043" H 4350 2300 50  0001 C CNN
 F 1 "GND" H 4350 2400 50  0000 C CNN
 F 2 "" H 4350 2550 50  0000 C CNN
@@
 	8850 2300 8850 2450
 Connection ~ 8850 2450
+Wire Wire Line
+	9650 1050 9650 1250
+$Comp
+L 74LS245 U8
+U 1 1 586E215C
+P 9650 1800
+F 0 "U8" H 9750 2375 50  0000 L BNN
+F 1 "74LS245" H 9700 1225 50  0000 L TNN
+F 2 "Housings_DIP:DIP-20_W7.62mm_LongPads" H 9650 1800 50  0001 C CNN
+F 3 "" H 9650 1800 50  0000 C CNN
+	1    9650 1800
+	1    0    0    -1
+$EndComp
 $EndSCHEMATC

Commit message: fixed up some footprint issues
Parts:
- P11: footprint Pin_Headers:Pin_Header_Straight_2x06_Pitch2.54mm -> Pin_Headers:Pin_Header_Straight_2x07_Pitch2.54mm
Changed lines of the file:
@@
 F 0 "P11" H 1500 1350 50  0000 C CNN
 F 1 "gui140x16j-7002" V 1500 950 50  0000 C CNN
-F 2 "Pin_Headers:Pin_Header_Straight_2x06_Pitch2.54mm" H 1500 -250 50  0001 C CNN
+F 2 "Pin_Headers:Pin_Header_Straight_2x07_Pitch2.54mm" H 1500 -250 50  0001 C CNN
 F 3 "" H 1500 -250 50  0000 C CNN
 	1    1500 950
