File: ac/bela-ac.kicad_pcb (KiCad board)
At the start: 2 copper layers, 31.8 x 69.9 mm, 34 parts, among them P5 +/-15v, P6 15v_out, P7 belaaudioout, P8 belaaudioin, P9 mod_ac-io, U1 TL074

Commit message: got the correct part in, AND the mounting holes
Parts:
- removed R17, R18: 2k, xnorman:Resistor_Horizontal_RM10mm-xnorman
- added R19: 1k, xnorman:Resistor_Horizontal_RM10mm-xnorman, F.Cu at (38.0, 129.2)
- added R20: 1k, xnorman:Resistor_Horizontal_RM10mm-xnorman, F.Cu at (38.0, 132.3)
Routing:
- net belaacin1: track 27.2 -> 2.54 mm
- net Net-(R11-Pad2): track 36.2 -> 19.0 mm
- net Net-(R15-Pad1): track 9.79 -> 0.00 mm
- net Net-(R16-Pad1): track 9.76 -> 0.00 mm
- net belaacin2: track 16.3 -> 12.1 mm
